File: PCB/board.brd (EAGLE design)
At the start: 35 x 50 mm, 10 parts, among them J1 PROG-HEADER_2X3_SHROUDED, J10 PROG-HEADER_2X5_1.27MM-PTH+SMD, J2 PROG-HEADER_2X5_2.00MM-SHROUD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, J3 PROG-HEADER_2X5_SHROUDED, J5 PROG-HEADER_2X10_RIGHT-ANGLE, J6 PROG-HEADER_2X10_SHROUDED, J8 CONN-1X4, J9 CONN-1X6

Commit message: V1
Parts:
- moved JP1 1.78 mm to (23.4, 26.4)
Routing:
- net VCC: track 0.00 -> 135.2 mm, vias 0 -> 1
- net TCK: track 0.00 -> 127.6 mm
- net RST: track 0.00 -> 98.7 mm, vias 0 -> 1
- net TMS: track 0.00 -> 97.1 mm, vias 0 -> 1
- net TDO: track 0.00 -> 87.6 mm
- net TDI: track 0.00 -> 74.7 mm
- net RTCK: track 0.00 -> 72.6 mm, vias 0 -> 1
- net 2: track 0.00 -> 28.9 mm
- net NTRST: track 0.00 -> 20.8 mm
Other:
- board text added: ">GITHUB"

Commit message: V1.1
Parts:
- moved J5 1.52 mm to (18.5, 4.06)
- moved J6 0.25 mm to (18.5, 14.0)
Routing:
- net TDI: track 74.7 -> 70.2 mm, vias 0 -> 1
- net NTRST: track 20.8 -> 24.2 mm
- net TCK: track 127.6 -> 130.7 mm
- net RST: track 98.7 -> 100.1 mm
- net TDO: track 87.6 -> 88.4 mm
- net 2: track 28.9 -> 29.6 mm
- net TMS: track 97.1 -> 97.8 mm
- net RTCK: track 72.6 -> 72.2 mm, vias 1 -> 2

Commit message: V1.2
Parts:
- removed JP2: (no value), pinhead_v2:1X06/OCT
- J10: value PROG-HEADER_2X5_1.27MM-PTH+SMD -> PROG-HEADER_2X5_1.27MM-SHROUDED_PTH_SMD; device angrypig7-Connectors-Programming:2X5-1.27MM_PTH+SMD -> angrypig7-Connectors-Programming:2X5-1.27MM-SHROUDED_PTH+SMD
- moved J2 8.10 mm to (4.83, 39.4), turned to 180 degrees
- moved J1 5.21 mm to (13.5, 39.1), turned to 0 degrees
- moved J10 1.27 mm to (23.4, 41.4), turned to 270 degrees
- moved J9 0.51 mm to (31.1, 34.0)
- moved J6 0.25 mm to (18.5, 13.7), turned to 90 degrees
- moved J5 0.25 mm to (18.5, 3.81)
Connections:
- net GND: no longer JP2.3
- net RST: no longer JP2.5
- net TCK: no longer JP2.2
- net TDO: no longer JP2.6
- net TMS: no longer JP2.4
- net VCC: no longer JP2.1
Routing:
- net TCK: track 130.7 -> 95.8 mm, vias 0 -> 2
- net NTRST: track 24.2 -> 7.42 mm
- net 2: track 29.6 -> 13.5 mm
- net TDO: track 88.4 -> 102.5 mm, vias 0 -> 1
- net VCC: track 134.8 -> 127.1 mm, vias 1 -> 0
- net RST: track 100.1 -> 95.3 mm, vias 1 -> 0
- net TMS: track 97.8 -> 94.0 mm, vias 1 -> 2
- net RTCK: track 72.2 -> 74.7 mm
- net TDI: track 70.2 -> 68.5 mm, vias 1 -> 0
