File: PCB/board.sch (EAGLE design)
At the start: 10 parts, among them J1 PROG-HEADER_2X3_SHROUDED, J10 PROG-HEADER_2X5_1.27MM-PTH+SMD, J2 PROG-HEADER_2X5_2.00MM-SHROUD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, J3 PROG-HEADER_2X5_SHROUDED, J5 PROG-HEADER_2X10_RIGHT-ANGLE, J6 PROG-HEADER_2X10_SHROUDED, J8 CONN-1X4, J9 CONN-1X6

Commit message: V1.1
Changed lines of the file:
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@@
 <schematic xreflabel="%F%N/%S.%C%R" xrefpart="/%S.%C%R">
 <attributes>
-<attribute name="CNAME" value="JTAG adapter"/>
-<attribute name="CREVISION" value="V1"/>
+<attribute name="CNAME" value="JTAG adapter board"/>
+<attribute name="CREVISION" value="V1.1"/>
 </attributes>
 <variantdefs>
@@
     (not required)
 RST: active low, target CPU reset signal</text>
+<text x="185.42" y="20.32" size="2.54" layer="94" font="vector">&gt;CNAME</text>
+<text x="237.49" y="5.08" size="2.54" layer="94" font="vector">&gt;CREVISION</text>
 </plain>
 <instances>

Commit message: V1.2
Parts:
- removed JP2: (no value), pinhead_v2:PINHD-1X6/OCT
- J10: value PROG-HEADER_2X5_1.27MM-PTH+SMD -> PROG-HEADER_2X5_1.27MM-SHROUDED_PTH_SMD; device angrypig7-Connectors-Programming:PROG-HEADER_2X5_1.27MM-PTH+SMD -> angrypig7-Connectors-Programming:PROG-HEADER_2X5_1.27MM-SHROUDED_PTH_SMD
Connections:
- net GND: no longer JP2.3
- net RST: no longer JP2.5
- net TCK: no longer JP2.2
- net TDO: no longer JP2.6
- net TMS: no longer JP2.4
- net VCC: no longer JP2.1
Changed lines of the file:
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@@
 <setting verticaltext="up"/>
 </settings>
-<grid distance="50" unitdist="mil" unit="mil" style="lines" multiple="1" display="no" altdistance="0.01" altunitdist="inch" altunit="inch"/>
+<grid distance="0.1" unitdist="inch" unit="inch" style="lines" multiple="1" display="no" altdistance="0.01" altunitdist="inch" altunit="inch"/>
 <layers>
 <layer number="1" name="Top" color="4" fill="1" visible="no" active="no"/>
@@
 <attributes>
 <attribute name="CNAME" value="JTAG adapter board"/>
-<attribute name="CREVISION" value="V1.1"/>
+<attribute name="CREVISION" value="V1.2"/>
 </attributes>
 <variantdefs>
@@
 <part name="J9" library="angrypig7-Connectors-Programming" deviceset="CONN-1X6" device=""/>
 <part name="JP1" library="SparkFun-Jumpers" deviceset="JUMPER-SMT_2_NO" device="_SILK" package3d_urn="urn:adsk.eagle:package:39279/1" value="TCK-RTCK"/>
-<part name="J10" library="angrypig7-Connectors-Programming" deviceset="PROG-HEADER_2X5" device="_1.27MM-PTH+SMD"/>
+<part name="J10" library="angrypig7-Connectors-Programming" deviceset="PROG-HEADER_2X5" device="_1.27MM-SHROUDED_PTH_SMD" value="PROG-HEADER_2X5_1.27MM-SHROUDED_PTH_SMD"/>
 <part name="J2" library="angrypig7-Connectors-Programming" deviceset="PROG-HEADER_2X5" device="_2.00MM-SHROUDED"/>
 <part name="J5" library="angrypig7-Connectors-Programming" deviceset="PROG-HEADER_2X10" device="_RIGHT-ANGLE"/>
-<part name="JP2" library="pinhead_v2" deviceset="PINHD-1X6" device="/OCT"/>
 </parts>
 <sheets>
@@
 <attribute name="VALUE" x="132.08" y="108.204" size="1.778" layer="96" font="vector"/>
 </instance>
-<instance part="JP2" gate="A" x="224.79" y="114.3" smashed="yes">
-<attribute name="NAME" x="218.44" y="125.095" size="1.778" layer="95"/>
-<attribute name="VALUE" x="218.44" y="104.14" size="1.778" layer="96"/>
-</instance>
 </instances>
 <busses>
@@
 <label x="207.01" y="121.92" size="1.27" layer="95" xref="yes"/>
 <pinref part="J9" gate="G$1" pin="1"/>
-<pinref part="JP2" gate="A" pin="1"/>
-<wire x1="222.25" y1="121.92" x2="201.93" y2="121.92" width="0.1524" layer="91"/>
+<wire x1="207.01" y1="121.92" x2="201.93" y2="121.92" width="0.1524" layer="91"/>
 </segment>
 <segment>
@@
 <label x="207.01" y="114.3" size="1.27" layer="95" xref="yes"/>
 <pinref part="J9" gate="G$1" pin="4"/>
-<pinref part="JP2" gate="A" pin="4"/>
-<wire x1="201.93" y1="114.3" x2="222.25" y2="114.3" width="0.1524" layer="91"/>
+<wire x1="201.93" y1="114.3" x2="207.01" y2="114.3" width="0.1524" layer="91"/>
 </segment>
 </net>
@@
 <label x="207.01" y="109.22" size="1.27" layer="95" xref="yes"/>
 <pinref part="J9" gate="G$1" pin="6"/>
-<pinref part="JP2" gate="A" pin="6"/>
-<wire x1="201.93" y1="109.22" x2="222.25" y2="109.22" width="0.1524" layer="91"/>
+<wire x1="201.93" y1="109.22" x2="207.01" y2="109.22" width="0.1524" layer="91"/>
 </segment>
 </net>
@@
 <label x="207.01" y="111.76" size="1.27" layer="95" xref="yes"/>
 <pinref part="J9" gate="G$1" pin="5"/>
-<pinref part="JP2" gate="A" pin="5"/>
-<wire x1="201.93" y1="111.76" x2="222.25" y2="111.76" width="0.1524" layer="91"/>
+<wire x1="201.93" y1="111.76" x2="207.01" y2="111.76" width="0.1524" layer="91"/>
 </segment>
 </net>
@@
 <label x="207.01" y="116.84" size="1.27" layer="95" xref="yes"/>
 <pinref part="J9" gate="G$1" pin="3"/>
-<pinref part="JP2" gate="A" pin="3"/>
-<wire x1="222.25" y1="116.84" x2="201.93" y2="116.84" width="0.1524" layer="91"/>
+<wire x1="207.01" y1="116.84" x2="201.93" y2="116.84" width="0.1524" layer="91"/>
 </segment>
 </net>
@@
 <label x="207.01" y="119.38" size="1.27" layer="95" xref="yes"/>
 <pinref part="J9" gate="G$1" pin="2"/>
-<pinref part="JP2" gate="A" pin="2"/>
-<wire x1="201.93" y1="119.38" x2="222.25" y2="119.38" width="0.1524" layer="91"/>
-</segment>
-</net>
+<wire x1="201.93" y1="119.38" x2="207.01" y2="119.38" width="0.1524" layer="91"/>
+</segment>
+</net>
