File: PCB/board.sch (EAGLE design)
At the start: 9 parts, among them J1 PROG-HEADER_2X3_SHROUDED, J10 PROG-HEADER_2X5_1.27MM-SHROUD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, J2 PROG-HEADER_2X5_2.00MM-SHROUD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, J3 PROG-HEADER_2X5_SHROUDED, J4 PROG-HEADER_2X10_2.54MM-END-L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, J6 PROG-HEADER_2X10_SHROUDED, J8 CONN-1X4, J9 CONN-1X6

Commit message: rollback to V1.4
Parts:
- JP1: device angrypig7-Jumpers:JUMPER-SMT_2_NO_SILK -> SparkFun-Jumpers:JUMPER-SMT_2_NO_SILK
Connections:
- net VREF renamed VCC
- removed net 17: J4.17, J6.17
- removed net 19: J4.19, J6.19
- removed net 2: J4.2, J6.2
- net RST: now also J1.3
- net TDI: no longer J1.3
Changed lines of the file:
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@@
 <?xml version="1.0" encoding="utf-8"?>
 <!DOCTYPE eagle SYSTEM "eagle.dtd">
-<eagle version="9.6.2">
+<eagle version="9.6.1">
 <drawing>
 <settings>
@@
 <attributes>
 <attribute name="CNAME" value="JTAG adapter board"/>
-<attribute name="CREVISION" value="V1.5"/>
+<attribute name="CREVISION" value="V1.4"/>
 </attributes>
 <variantdefs>
@@
 <part name="J8" library="angrypig7-Connectors-Programming" deviceset="CONN-1X4" device=""/>
 <part name="J9" library="angrypig7-Connectors-Programming" deviceset="CONN-1X6" device=""/>
-<part name="JP1" library="angrypig7-Jumpers" deviceset="JUMPER-SMT_2_NO" device="_SILK" package3d_urn="urn:adsk.eagle:package:39279/1" value="TCK-RTCK"/>
+<part name="JP1" library="SparkFun-Jumpers" deviceset="JUMPER-SMT_2_NO" device="_SILK" package3d_urn="urn:adsk.eagle:package:39279/1" value="TCK-RTCK"/>
 <part name="J10" library="angrypig7-Connectors-Programming" deviceset="PROG-HEADER_2X5" device="_1.27MM-SHROUDED_PTH_SMD" value="PROG-HEADER_2X5_1.27MM-SHROUDED_PTH_SMD"/>
 <part name="J2" library="angrypig7-Connectors-Programming" deviceset="PROG-HEADER_2X5" device="_2.00MM-SHROUDED"/>
@@
 </instance>
 <instance part="J1" gate="G$1" x="63.5" y="143.51" smashed="yes">
-<attribute name="NAME" x="59.69" y="149.098" size="1.778" layer="95" font="vector"/>
+<attribute name="NAME" x="57.15" y="149.098" size="1.778" layer="95" font="vector"/>
 <attribute name="VALUE" x="57.15" y="136.144" size="1.778" layer="96" font="vector"/>
 </instance>
@@
 </instance>
 <instance part="J8" gate="G$1" x="196.85" y="139.7" smashed="yes">
-<attribute name="VALUE" x="196.85" y="131.064" size="1.778" layer="96" font="vector"/>
-<attribute name="NAME" x="196.85" y="146.558" size="1.778" layer="95" font="vector"/>
+<attribute name="VALUE" x="191.77" y="132.334" size="1.778" layer="96" font="vector"/>
+<attribute name="NAME" x="191.77" y="147.828" size="1.778" layer="95" font="vector"/>
 </instance>
 <instance part="J9" gate="G$1" x="196.85" y="114.3" smashed="yes">
-<attribute name="VALUE" x="196.85" y="103.124" size="1.778" layer="96" font="vector"/>
-<attribute name="NAME" x="196.85" y="123.698" size="1.778" layer="95" font="vector"/>
+<attribute name="VALUE" x="191.77" y="104.394" size="1.778" layer="96" font="vector"/>
+<attribute name="NAME" x="191.77" y="124.968" size="1.778" layer="95" font="vector"/>
 </instance>
 <instance part="JP1" gate="G$1" x="152.4" y="11.43" smashed="yes">
@@
 </busses>
 <nets>
-<net name="VREF" class="0">
+<net name="VCC" class="0">
 <segment>
 <wire x1="54.61" y1="128.27" x2="49.53" y2="128.27" width="0.1524" layer="91"/>
@@
 </segment>
 <segment>
-<wire x1="204.47" y1="135.89" x2="207.01" y2="135.89" width="0.1524" layer="91"/>
-<label x="207.01" y="135.89" size="1.27" layer="95" xref="yes"/>
+<wire x1="204.47" y1="135.89" x2="207.01" y2="137.16" width="0.1524" layer="91"/>
+<label x="207.01" y="137.16" size="1.27" layer="95" xref="yes"/>
 <pinref part="J8" gate="G$1" pin="4"/>
 </segment>
 <segment>
-<label x="207.01" y="120.65" size="1.27" layer="95" xref="yes"/>
+<label x="207.01" y="121.92" size="1.27" layer="95" xref="yes"/>
 <pinref part="J9" gate="G$1" pin="1"/>
-<wire x1="207.01" y1="120.65" x2="204.47" y2="120.65" width="0.1524" layer="91"/>
+<wire x1="207.01" y1="121.92" x2="204.47" y2="120.65" width="0.1524" layer="91"/>
 </segment>
 <segment>
@@
 </segment>
 <segment>
-<wire x1="204.47" y1="138.43" x2="207.01" y2="138.43" width="0.1524" layer="91"/>
-<label x="207.01" y="138.43" size="1.27" layer="95" xref="yes"/>
+<wire x1="204.47" y1="138.43" x2="207.01" y2="139.7" width="0.1524" layer="91"/>
+<label x="207.01" y="139.7" size="1.27" layer="95" xref="yes"/>
 <pinref part="J8" gate="G$1" pin="3"/>
 </segment>
@@
 </segment>
 <segment>
-<label x="207.01" y="113.03" size="1.27" layer="95" xref="yes"/>
+<label x="207.01" y="114.3" size="1.27" layer="95" xref="yes"/>
 <pinref part="J9" gate="G$1" pin="4"/>
-<wire x1="204.47" y1="113.03" x2="207.01" y2="113.03" width="0.1524" layer="91"/>
+<wire x1="204.47" y1="113.03" x2="207.01" y2="114.3" width="0.1524" layer="91"/>
 </segment>
 </net>
@@
 </segment>
 <segment>
-<label x="207.01" y="107.95" size="1.27" layer="95" xref="yes"/>
+<label x="207.01" y="109.22" size="1.27" layer="95" xref="yes"/>
 <pinref part="J9" gate="G$1" pin="6"/>
-<wire x1="204.47" y1="107.95" x2="207.01" y2="107.95" width="0.1524" layer="91"/>
+<wire x1="204.47" y1="107.95" x2="207.01" y2="109.22" width="0.1524" layer="91"/>
 </segment>
 </net>
@@
 <pinref part="J4" gate="G$1" pin="5"/>
 </segment>
+</net>
+<net name="RST" class="0">
+<segment>
+<wire x1="72.39" y1="118.11" x2="77.47" y2="118.11" width="0.1524" layer="91"/>
+<label x="77.47" y="118.11" size="1.27" layer="95" xref="yes"/>
+<pinref part="J3" gate="G$1" pin="10"/>
+</segment>
+<segment>
+<wire x1="127" y1="80.01" x2="121.92" y2="80.01" width="0.1524" layer="91"/>
+<label x="121.92" y="80.01" size="1.27" layer="95" rot="R180" xref="yes"/>
+<pinref part="J6" gate="G$1" pin="15"/>
+</segment>
 <segment>
 <wire x1="54.61" y1="143.51" x2="49.53" y2="143.51" width="0.1524" layer="91"/>
@@
 <pinref part="J1" gate="G$1" pin="3"/>
 </segment>
-</net>
-<net name="RST" class="0">
-<segment>
-<wire x1="72.39" y1="118.11" x2="77.47" y2="118.11" width="0.1524" layer="91"/>
-<label x="77.47" y="118.11" size="1.27" layer="95" xref="yes"/>
-<pinref part="J3" gate="G$1" pin="10"/>
-</segment>
-<segment>
-<wire x1="127" y1="80.01" x2="121.92" y2="80.01" width="0.1524" layer="91"/>
-<label x="121.92" y="80.01" size="1.27" layer="95" rot="R180" xref="yes"/>
-<pinref part="J6" gate="G$1" pin="15"/>
-</segment>
 <segment>
 <wire x1="72.39" y1="92.71" x2="77.47" y2="92.71" width="0.1524" layer="91"/>
@@
 </segment>
 <segment>
-<label x="207.01" y="110.49" size="1.27" layer="95" xref="yes"/>
+<label x="207.01" y="111.76" size="1.27" layer="95" xref="yes"/>
 <pinref part="J9" gate="G$1" pin="5"/>
-<wire x1="204.47" y1="110.49" x2="207.01" y2="110.49" width="0.1524" layer="91"/>
+<wire x1="204.47" y1="110.49" x2="207.01" y2="111.76" width="0.1524" layer="91"/>
 </segment>
 </net>
@@
 </segment>
 <segment>
-<wire x1="204.47" y1="143.51" x2="207.01" y2="143.51" width="0.1524" layer="91"/>
-<label x="207.01" y="143.51" size="1.27" layer="95" xref="yes"/>
+<wire x1="204.47" y1="143.51" x2="207.01" y2="144.78" width="0.1524" layer="91"/>
+<label x="207.01" y="144.78" size="1.27" layer="95" xref="yes"/>
 <pinref part="J8" gate="G$1" pin="1"/>
 </segment>
@@
 </segment>
 <segment>
-<label x="207.01" y="115.57" size="1.27" layer="95" xref="yes"/>
+<label x="207.01" y="116.84" size="1.27" layer="95" xref="yes"/>
 <pinref part="J9" gate="G$1" pin="3"/>
-<wire x1="207.01" y1="115.57" x2="204.47" y2="115.57" width="0.1524" layer="91"/>
+<wire x1="207.01" y1="116.84" x2="204.47" y2="115.57" width="0.1524" layer="91"/>
 </segment>
 <segment>
@@
 <net name="TCK" class="0">
 <segment>
-<wire x1="204.47" y1="140.97" x2="207.01" y2="140.97" width="0.1524" layer="91"/>
-<label x="207.01" y="140.97" size="1.27" layer="95" xref="yes"/>
+<wire x1="204.47" y1="140.97" x2="207.01" y2="142.24" width="0.1524" layer="91"/>
+<label x="207.01" y="142.24" size="1.27" layer="95" xref="yes"/>
 <pinref part="J8" gate="G$1" pin="2"/>
 </segment>
@@
 </segment>
 <segment>
-<label x="207.01" y="118.11" size="1.27" layer="95" xref="yes"/>
+<label x="207.01" y="119.38" size="1.27" layer="95" xref="yes"/>
 <pinref part="J9" gate="G$1" pin="2"/>
-<wire x1="204.47" y1="118.11" x2="207.01" y2="118.11" width="0.1524" layer="91"/>
+<wire x1="204.47" y1="118.11" x2="207.01" y2="119.38" width="0.1524" layer="91"/>
 </segment>
 </net>
@@
 </segment>
 </net>
-<net name="2" class="0">
-<segment>
-<pinref part="J4" gate="G$1" pin="2"/>
-<wire x1="144.78" y1="135.89" x2="149.86" y2="135.89" width="0.1524" layer="91"/>
-<label x="149.86" y="135.89" size="1.27" layer="95" xref="yes"/>
-</segment>
-<segment>
-<pinref part="J6" gate="G$1" pin="2"/>
-<wire x1="144.78" y1="97.79" x2="149.86" y2="97.79" width="0.1524" layer="91"/>
-<label x="149.86" y="97.79" size="1.27" layer="95" xref="yes"/>
-</segment>
-</net>
-<net name="17" class="0">
-<segment>
-<pinref part="J6" gate="G$1" pin="17"/>
-<wire x1="127" y1="77.47" x2="121.92" y2="77.47" width="0.1524" layer="91"/>
-<label x="121.92" y="77.47" size="1.27" layer="95" rot="R180" xref="yes"/>
-</segment>
-<segment>
-<pinref part="J4" gate="G$1" pin="17"/>
-<wire x1="127" y1="115.57" x2="121.92" y2="115.57" width="0.1524" layer="91"/>
-<label x="121.92" y="115.57" size="1.27" layer="95" rot="R180" xref="yes"/>
-</segment>
-</net>
-<net name="19" class="0">
-<segment>
-<pinref part="J6" gate="G$1" pin="19"/>
-<wire x1="127" y1="74.93" x2="121.92" y2="74.93" width="0.1524" layer="91"/>
-<label x="121.92" y="74.93" size="1.27" layer="95" rot="R180" xref="yes"/>
-</segment>
-<segment>
-<pinref part="J4" gate="G$1" pin="19"/>
-<wire x1="127" y1="113.03" x2="121.92" y2="113.03" width="0.1524" layer="91"/>
-<label x="121.92" y="113.03" size="1.27" layer="95" rot="R180" xref="yes"/>
-</segment>
-</net>

Commit message: V1.6 update
Parts:
- removed J2: PROG-HEADER_2X5_2.00MM-SHROUDED, angrypig7-Connectors-Programming:PROG-HEADER_2X5_2.00MM-SHROUDED
- removed J6: PROG-HEADER_2X10_SHROUDED, angrypig7-Connectors-Programming:PROG-HEADER_2X10_SHROUDED
- removed J9: CONN-1X6, angrypig7-Connectors-Programming:CONN-1X6
- removed JP1: TCK-RTCK, SparkFun-Jumpers:JUMPER-SMT_2_NO_SILK
- added C1: 100nF, angrypig7-RCL:C-NON-POLC0603
- added S1: SWITCH-SPST-SMD-5.1MM, angrypig7-Switches:SWITCH-SPST-SMD-5.1MM
Connections:
- net GND: now also C1.2, S1.2; no longer J2.3, J2.5, J2.9, J6.10, J6.12, J6.14, J6.16, J6.18, J6.20, J6.4, J6.6, J6.8, J9.3
- net NTRST: no longer J6.3
- net RST: now also C1.1, S1.1; no longer J2.10, J6.15, J9.5
- net RTCK: no longer J2.7, J6.11, JP1.2
- net TCK: no longer J2.4, J6.9, J9.2, JP1.1
- net TDI: no longer J2.8, J6.5
- net TDO: no longer J2.6, J6.13, J9.6
- net TMS: no longer J2.2, J6.7, J9.4
- net VCC: no longer J2.1, J6.1, J9.1
